File: Design Reference/Sample CAN Breakout/Sample CAN Breakout.kicad_sch (KiCad schematic)
At the start: 7 parts, among them J1 2604-1102, J2 2604-1102, J3 2604-1102, J4 2604-1102, J5 2604-1102, J6 2604-1102, J7 2604-1102

Commit message: Reference Design 1 Finished
Ruler Reference Design Finished
Other:
- company: (none) -> FRC Team 619
- title: (none) -> CAN Bus Breakout Reference Schematic
Changed lines of the file:
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@@
 (kicad_sch (version 20211123) (generator eeschema)
   (paper "A4")
+  (title_block
+    (title "CAN Bus Breakout Reference Schematic")
+    (date "2023-01-12")
+    (rev "1")
+    (company "FRC Team 619")
+  )
   (junction (at 160.02 99.06) (diameter 0) (color 0 0 0 0)
   )
